Commit message: update system

File: assets/bike_v3.urdf (robot description, URDF)
Before this commit: robot bike_V3_urdf, 5 links, 4 joints
Links:
- removed link world
- added link imu_link, mass 0.000001
Joints:
- removed joint floating_base
- added joint imu_fixed: type fixed, parent main_body, child imu_link, origin xyz=-0.200000 0 0.424357 rpy=0 0 0
- joint fork_yaw: limit lower=-1.570796 upper=1.570796 effort=12.0 velocity=100.0 -> lower=-1.570796 upper=1.570796; origin xyz=-0.492314 0 0.34492 rpy=0 0.20847 -0 -> xyz=-0.492314 0 0.34492 rpy=0 0.20847 0
